File: HC Macropad MCU.kicad_sch (KiCad schematic)
At the start: 36 parts, among them J1 USB_C_Receptacle_USB2.0_16P, J2 Conn_01x02_Socket, J3 Conn_01x04_Socket, SW1 SW_Push, U1 RP2040, U2 W25Q128JVPIQ, U3 AP2127K-3.3, U4 USBLC6-2P6, Y1 Crystal_GND24

Commit message: 90% of routing done
Parts:
- added J4, J5: Conn_01x04_Socket, Connector_PinHeader_2.54mm:PinHeader_1x04_P2.54mm_Vertical, symbol Connector:Conn_01x04_Socket
Connections:
- net +5V: now also J4.1 (Pin_1), J5.1 (Pin_1)
- net D+: now also J4.3 (Pin_3), J5.3 (Pin_3)
- net D-: now also J4.2 (Pin_2), J5.2 (Pin_2)
- net ENC_PIN0: now also U1.14 (GPIO11); no longer U1.12 (GPIO9)
- net ENC_SW0: now also U1.11 (GPIO8); no longer U1.14 (GPIO11)
- net ENC_SW1: now also U1.12 (GPIO9); no longer U1.15 (GPIO12)
- net GND: now also J4.4 (Pin_4), J5.4 (Pin_4)
- net M_COL0: now also U1.38 (GPIO26_ADC0); no longer U1.8 (GPIO6)
- net M_COL1: now also U1.39 (GPIO27_ADC1); no longer U1.9 (GPIO7)
- net M_COL2: now also U1.40 (GPIO28_ADC2); no longer U1.11 (GPIO8)
- net M_ROW0: now also U1.37 (GPIO25); no longer U1.6 (GPIO4)
- net M_ROW1: now also U1.36 (GPIO24); no longer U1.7 (GPIO5)
