File: HC Macropad MCU.kicad_sch (KiCad schematic)
At the start: 38 parts, among them J1 USB_C_Receptacle_USB2.0_16P, J2 Conn_01x02_Socket, J3 Conn_01x04_Socket, J4 Conn_01x04_Socket, J5 Conn_01x04_Socket, SW1 SW_Push, U1 RP2040, U2 W25Q128JVPIQ, U3 AP2127K-3.3, U4 USBLC6-2P6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

Commit message: v0.1.3: UFE edition
Parts:
- J2, J3, J4, J5: now left out of the parts list
Changed lines of the file:
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@@
 		(title "HC Macropad")
 		(date "2024-10-07")
-		(rev "0.1.2")
+		(rev "0.1.3")
 		(company "Google")
 		(comment 1 "Licensed under CERN-OHL-W v2")
@@
 		(unit 1)
 		(exclude_from_sim no)
-		(in_bom yes)
+		(in_bom no)
 		(on_board yes)
 		(dnp no)
@@
 		(unit 1)
 		(exclude_from_sim no)
-		(in_bom yes)
+		(in_bom no)
 		(on_board yes)
 		(dnp no)
@@
 		(unit 1)
 		(exclude_from_sim no)
-		(in_bom yes)
+		(in_bom no)
 		(on_board yes)
 		(dnp no)
@@
 		(unit 1)
 		(exclude_from_sim no)
-		(in_bom yes)
+		(in_bom no)
 		(on_board yes)
 		(dnp no)
